File: FastDataAcq.sch (EAGLE design)
At the start: 221 parts, among them J1 MICRO-FIT_3.0_2POS_RA_SMD, J2 USB_MICROAB_SMT, U1 ADC08D500, U10 TMP421, U11 DAC101C081, U12 ADCMP553BRMZ, U13 XCFXXS04, U14 FT230XQ, U2 XC6SLX9-3TQG144C, U3 LTC2955-1, U4 LT1963AEST-2.5, U5 LT1963AEST-3.3, U6 LT1963AEQ, U7 LTC3374QFN, U8 LMH6555, U9 LMV321SC-70, X1 SMA-142-0701-801/806, X2 SMA-142-0701-801/806, X3 HEADER_0.1"_8P_2R_SMT, X4 87832-14, Y1 SI530-500, Y2 100MHz, Y3 DNP

Commit message: PCB Power Layer and Other Fixes
Finalized the FPGA GPIO Pins. Fixed power layer so that all spacing is
equal and entire layer covered. Other cosmetic fixes.

Conflicts:
	FastDataAcq.brd
	FastDataAcq.sch
	To Do List
	eagle.epf
Parts:
- removed C7: .1uF, Schuyler:CAPACITOR0204_REVERSE
- removed PAD1, PAD2, PAD3, PAD4: (no value), wirepad:SMD2
- removed R26: DNP, rcl:R-US_R0603
- removed TP1, TP2: TEST-POINT3, SparkFun-Passives:TEST-POINT3
- removed U3: LTC2955-1, Schuyler:LTC2955-1
- added U$14: LTC2955-1, Schuyler:LTC2955-1
- C30: value 33uF -> .1uF; device SparkFun-Passives:CAP0805 -> Schuyler:CAPACITOR0204_REVERSE; PARTNUMBER 445-8238-1-ND -> 587-2152-1-ND; SUPPLIER (none) -> DIGIKEY
- R40: value 50 -> DNP; device rcl:R-US_R0201 -> rcl:R-US_R0603; MANPARTNUMBER RC0603F49R9C -> (none); MANUFACTURER Samsung Electro-Mechanics America, Inc -> (none); PARTNUMBER 1276-3590-1-ND -> 311-0.0GRCT-ND
- renumbered X3 to U$95
Connections:
- net !PB: no longer U3.!PB
- net 1V9A: now also R6.1, R8.2; no longer R3.1, R6.2, U1G$1.VA@11
- net 2V5: now also L11.P$2; no longer L12.P$2
- net 2V5A: now also C76.1, C77.1, C78.1, L11.P$1; no longer C85.1, C86.1, C87.1, L12.P$1
- net 3V3: now also C80.1, C81.1, R42.1; no longer C102.1, C104.1, R45.1, U13.VCCINT, U13.VCCJ, U13.VCCO
- net ADC_CAL: now also R6.2; no longer R3.2, U1G$1.CAL
- net ADC_CLK_N: no longer U1G$1.CLK-
- net ADC_CLK_P: no longer U1G$1.CLK+
- net ADC_OUTEDGE/DDR/SDATA: no longer U1G$1.OUTEDGE/DDR/SDATA
- net ADC_PD: no longer U1G$1.PD
- net ADC_REXT: now also R9.2; no longer R7.2, U1G$1.REXT
- net ADC_VBG: now also R8.1; no longer R6.1, U1G$1.VBG
- net ADC_VCMO: no longer U1G$1.VCMO
- net ADC_VCMO_BUFFER: no longer U1G$1.VINQ+, U1G$1.VINQ-
- net ADC_VINI+: no longer U1G$1.VINI+
- net ADC_VINI-: no longer U1G$1.VINI-
- net GND: now also C77.2, C78.2, R9.1; no longer C102.2, C104.2, C7.2, C85.2, C86.2, C87.2, PAD1.P, PAD2.P, PAD3.P, PAD4.P, R7.1, U2.GND@7, U3.GND, U3.PAD
- net N$12: no longer U3.ON
- net N$17: no longer U3.TMR
- net PWR_ENABLE: no longer TP2.1, U3.EN
- net PWR_INT: no longer U3.!INT
- net PWR_KILL: no longer U3.!KILL
- net S_MODE: no longer R26.2
- net TRIG_REF: no longer TP1.1
- net TRIG_RESET_HIGH: no longer U2.IO_L49N_D4_2
- net TRIG_RESET_LOW: no longer U2.IO_L49P_D3_2
- net VIN: no longer C7.1, R26.1, U3.SEL, U3.VIN
Other:
- moved on the sheet: C102, C30, C77, C78, C79, L11, L12, R2, R3, R6, R8, R9
