File: FastDataAcqSch.brd (EAGLE design)
At the start: 160 x 100 mm, 82 parts, among them IC2 IC_FT230X-SSOP-16, X1 SMA-SMDRA, X2 87832-14, Y1 SI530-500

Commit message: Update from end of day 8/31
Added USB/UART interface.

Conflicts:
	To Do List
	eagle.epf
Parts:
- removed IC2: IC_FT230X-SSOP-16, dp_devices:SSOP-16-FTDI
- added C56: 4.7uF, Schuyler:0306REVERSE
- added C57, C58: .1uF, Schuyler:0204REVERSE
- added C59, C60: 47pF, rcl:C0201
- added C61: 10nF, rcl:C0201
- added IC1: FT230XQ, ftdichip:QFN16
- added J1: USB_MICROAB_SMT, Schuyler:USB_MICROAB_SMT_1
- added L5: 600@100MHz, dp_devices:FB603
- added R15, R16: 27, rcl:R0201
- added R17, R18: 300, rcl:R0201
- C1, C10, C11, C12, C13, C14, C15, C16, C17, C18, C19, C2, C22, C26, C28, C29, C3, C4, C5, C54, C6, C7, C8, C9: value .1 uF -> .1uF
- C23, C55: value 1 uF -> 1uF
Connections:
- removed net 3V3OUT: IC2.10
- removed net VCCIO: IC2.3
- new net 5VUSB: C56.P$1, C57.P$2, IC1.10, L5.1
- new net 5VUSB_CON: C61.1, J1.VCC, L5.2
- new net FPGA_RXD: R17.2, U$2.P$41
- new net FPGA_TXD: R18.2, U$2.P$40
- new net FTDI_RXD: IC1.2, R18.1
- new net FTDI_TXD: IC1.15, R17.1
- new net N$3: IC1.6, R15.2
- new net N$4: C59.2, J1.D+, R15.1
- new net N$5: C60.2, J1.D-, R16.1
- new net N$7: IC1.7, R16.2
- new net N$8: C58.P$2, IC1.1, IC1.8, IC1.9
- net DGND: now also C56.P$2, C57.P$1, C58.P$1, C59.1, C60.1, C61.2, IC1.3, J1.GND
- net DQD5-: now also U$1.P$50
- net GND: now also IC1.13
Routing:
- net 1V8: track 0.00 -> 316.5 mm
- net ADC_PD: track 139.0 -> 0.00 mm
- net DQD5-: track 0.00 -> 133.8 mm
- net 1V9D: track 399.1 -> 266.7 mm
- net DQ5+: track 134.3 -> 15.3 mm
- net ADC_DCLK-: track 59.8 -> 9.07 mm
- net DI7+: track 135.0 -> 118.0 mm
- net DQD3-: track 133.8 -> 132.2 mm
- net DIO-: track 133.8 -> 132.3 mm
- net DID2-: track 135.3 -> 133.7 mm

Commit message: Added
Parts:
- removed R1: 50, rcl:R0402
- removed R9: NA, rcl:R0603
Connections:
- removed net FGPA_PROGRAMB: U$2.P$37
- removed net N$6: U$2.P$35
- net 1V2: now also C81.1, C90.1, L8.P$2, R34.2, R42.2, TP2.TP
- net 1V8: now also C83.1, C88.1, L7.P$2, R30.2, TP4.TP
- net 1V9: now also C94.1, IC2.4, R46.2, TP7.TP
- net 1V9A: now also R51.2; no longer R9.2
- net 2V5: now also C95.1, TP8.TP, U$9.3
- net 3V3: no longer L4.P$2
- net ADC_CALDLY/DES/!SCS: now also R51.1; no longer R9.1
- net AGND: no longer R1.2
- net N$2: now also R1.2; no longer R1.1
