File: FastDataAcqSch.sch (EAGLE design)
At the start: 82 parts, among them IC2 IC_FT230X-SSOP-16, X1 SMA-SMDRA, X2 87832-14, Y1 SI530-500

Commit message: Update from end of day 8/31
Added USB/UART interface.

Conflicts:
	To Do List
	eagle.epf
Parts:
- removed IC2: IC_FT230X-SSOP-16, dp_devices:IC_FT230X-SSOP-16
- added C56: 4.7uF, Schuyler:CAPACITOR0304_REVERSE
- added C57, C58: .1uF, Schuyler:CAPACITOR0204_REVERSE
- added C59, C60: 47pF, rcl:C-EUC0201
- added C61: 10nF, rcl:C-EUC0201
- added IC1: FT230XQ, ftdichip:FT230XQ
- added J1: USB_MICROAB_SMT, Schuyler:USB_MICROAB_SMT
- added L5: 600@100MHz, dp_devices:FERRITE-0603
- added R15, R16: 27, rcl:R-US_R0201
- added R17, R18: 300, rcl:R-US_R0201
- C1, C10, C11, C12, C13, C14, C15, C16, C17, C18, C19, C2, C22, C26, C28, C29, C3, C4, C5, C54, C6, C7, C8, C9: value .1 uF -> .1uF
- C23, C55: value 1 uF -> 1uF
Connections:
- new net 5VUSB: C56.1, C57.2, IC1.VCC, L5.1
- new net 5VUSB_CON: C61.1, J1.VCC, L5.2
- new net FPGA_RXD: R17.2, U$2.IO_L64P_D8_2
- new net FPGA_TXD: R18.2, U$2.IO_L64N_D9_2
- new net FTDI_RXD: IC1.RXD, R18.1
- new net FTDI_TXD: IC1.TXD, R17.1
- new net N$3: IC1.USBDP, R15.2
- new net N$4: C59.2, J1.D+, R15.1
- new net N$5: C60.2, J1.D-, R16.1
- new net N$7: IC1.USBDM, R16.2
- new net N$8: C58.2, IC1.!RESET, IC1.3V3OUT, IC1.VCCIO
- net DGND: now also C56.2, C57.1, C58.1, C59.1, C60.1, C61.2, IC1.GND, J1.GND
- net DQD5-: now also U$1.DQD5-
Other:
- note added: "Note: Current limiting resistors may not be necessary."

Commit message: Added
Parts:
- removed R1: 50, rcl:R-US_R0402
- removed R9: NA, rcl:R-US_R0603
Connections:
- net FGPA_PROGRAMB renamed FPGA_PROGRAMB
- removed net N$6: U$2.IO_L1P_3
- net 1V9A: no longer R9.2
- net ADC_CALDLY/DES/!SCS: no longer R9.1
- net AGND: no longer R1.2
- net N$2: no longer R1.1
Other:
- note added: "FPGA & Digital Power"
- note added: "NOTE: ADC is initially in Power Down mode (PD/PDQ pulled high) and calibration delayed (ADC_CAL pulled high). When the FPGA is ready, it can begin the ADC power and calibration process."
- note added: "Note: LDOs require >10mOhms ESR for stability and ringing damping."
- note added: "Note: Maybe make C bigger"
- note added: "Note: Ven is 420mV. Resistor divider should account for transient droop of at least 100mV."
- note added: "Power Regulation"
- note added: "Power Sequencing: 1) 1V2 supply is always enabled. 2) 3V3 enable once 1V2 is ready 3) 1V8 enabled once 3V3 is ready 4) ADC 1V9 enabled from FPGA 5) 2V5 and 3V3A enabled from FPGA. These shoud only be enabled after 1V9 is stable."
- moved on the sheet: C1, C10, C11, C12, C13, C14, C15, C16, C17, C18, C19, C2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

Commit message: Unchecked Finalized Schematic
Conflicts:
	FastDataAcqSch.brd
	FastDataAcqSch.sch
	To Do List
	eagle.epf
Parts:
- added D1, D6: LED_0603_RED, Schuyler:LED_0603_RED
- added D2, D5: LED_0603_GREEN, Schuyler:LED_0603_GREEN
- added D3, D4: LED_0603_BLUE, Schuyler:LED_0603_BLUE
- added H1, H2, H3, H4: MOUNT-HOLE2.8, holes:MOUNT-HOLE2.8
- added JP2: M10", SparkFun-Connectors:M10"
- added JP3: (no value), SparkFun-Passives:JUMPER-2PTH
- added L11: FERRITE_BEADS_BLM18SG331, Schuyler:FERRITE_BEADS_BLM18SG331
- added R23: 10k, rcl:R-US_R0201
- added R24: 1k, rcl:R-US_R0201
- added R56, R57, R58, R59, R60: 330, rcl:R-US_R0201
- added R61: 50, rcl:R-US_R0201
- added R62: NA, rcl:R-US_R0603
- added TP10, TP11, TP12, TP13, TP14, TP15: TPPAD1-13, testpad:TPPAD1-13
Connections:
- new net !RXLED: D2.CATHODE
- new net !TXLED: D3.CATHODE
- new net FPGA_GPIO0: JP2.1, U$2.IO_L49P_D3_2
- new net FPGA_GPIO1: JP2.2, U$2.IO_L14N_D12_2
- new net FPGA_GPIO2: JP2.3, U$2.IO_L14P_D11_2
- new net FPGA_GPIO3: JP2.4, U$2.IO_L13N_D10_2
- new net FPGA_GPIO4: JP2.5, U$2.IO_L12N_D2_MISO3_2
- new net FPGA_GPIO5: D6.CATHODE, JP2.6, U$2.IO_L12P_D1_MISO2_2
- new net FPGA_GPIO6: D5.CATHODE, JP2.7, U$2.IO_L3N_MOSI_CSI_B_MISO0_2
- new net FPGA_GPIO7: D4.CATHODE, JP2.8, U$2.IO_L2P_CMPCLK_2
- new net N$10: D2.ANODE, R56.2
- new net N$13: D3.ANODE, R57.2
- new net N$19: D6.ANODE, R60.2
- new net N$21: D5.ANODE, R59.2
- new net N$22: D4.ANODE, R58.2
- new net N$26: U$2.GND@10, U$2.GND@8, U$2.GND@9
- new net PGOOD: U$2.IO_L49N_D4_2
- new net S1SW: L11.P$1
- net 1V8: now also U$2.GND@7
- net 3V3: now also JP2.10, L11.P$2, R58.1, R59.1, R60.1, U$2.VCCAUX@4
Other:
- note added: "Power Sequencing: 1) 1V2 supply is always enabled. 2) 3V3 enable once 1V2 is ready 3) ADC 1V9 enabled from FPGA 4) 2V5 and 3V3A enabled from FPGA. These shoud only be enabled after 1V9 is stable."
- note removed: "Power Sequencing: 1) 1V2 supply is always enabled. 2) 3V3 enable once 1V2 is ready 3) 1V8 enabled once 3V3 is ready 4) ADC 1V9 enabled from FPGA 5) 2V5 and 3V3A enabled from FPGA. These shoud only be enabled after 1V9 is stable."
